Commit message: Add ground to train file

File: source/isaaclab_assets/isaaclab_assets/legged_v3/cad/robot.SLDASM/urdf/robot.SLDASM.urdf (robot description, URDF)
Before this commit: robot robot.SLDASM, 15 links, 16 joints
Links:
- link wheel_link_left: geometry collision cylinder length=0.045 radius=0.0765; visual mesh filename=../meshes/wheel_link_left.STL
- link wheel_link_right: geometry collision cylinder length=0.045 radius=0.0765; visual mesh filename=../meshes/wheel_link_right.STL
Joints:
- joint calf_joint_left_1: limit lower=-1.5708 upper=1.5708 effort=20 velocity=50 -> lower=-0.5 upper=0.5 effort=20 velocity=50
- joint calf_joint_left_2: limit lower=-1.5708 upper=1.5708 effort=0 velocity=50 -> lower=-0.5 upper=0.5 effort=0 velocity=50
- joint calf_joint_right_1: limit lower=-1.5708 upper=1.5708 effort=20 velocity=50 -> lower=-0.5 upper=0.5 effort=20 velocity=50
- joint calf_joint_right_2: limit lower=-1.5708 upper=1.5708 effort=0 velocity=50 -> lower=-0.5 upper=0.5 effort=0 velocity=50
- joint thigh_joint_left_1: limit lower=-1.5708 upper=1.5708 effort=20 velocity=50 -> lower=-0.5 upper=0.5 effort=20 velocity=50
- joint thigh_joint_left_2: limit lower=-1.5708 upper=1.5708 effort=0 velocity=50 -> lower=-0.5 upper=0.5 effort=0 velocity=50
- joint thigh_joint_right_1: limit lower=-1.5708 upper=1.5708 effort=20 velocity=50 -> lower=-0.5 upper=0.5 effort=20 velocity=50
- joint thigh_joint_right_2: limit lower=-1.5708 upper=1.5708 effort=0 velocity=50 -> lower=-0.5 upper=0.5 effort=0 velocity=50

Commit message: update param and func in vel

File: source/isaaclab_assets/isaaclab_assets/legged_v3/cad/robot.SLDASM/urdf/robot.SLDASM.urdf (robot description, URDF)
Before this commit: robot robot.SLDASM, 15 links, 16 joints
Joints:
- joint calf_joint_left_1: limit lower=-0.5 upper=0.5 effort=20 velocity=50 -> lower=-1.0 upper=1.0 effort=20 velocity=50
- joint calf_joint_left_2: limit lower=-0.5 upper=0.5 effort=0 velocity=50 -> lower=-1.0 upper=1.0 effort=0 velocity=50
- joint calf_joint_right_1: limit lower=-0.5 upper=0.5 effort=20 velocity=50 -> lower=-1.0 upper=1.0 effort=20 velocity=50
- joint calf_joint_right_2: limit lower=-0.5 upper=0.5 effort=0 velocity=50 -> lower=-1.0 upper=1.0 effort=0 velocity=50
- joint thigh_joint_left_1: limit lower=-0.5 upper=0.5 effort=20 velocity=50 -> lower=-1.0 upper=1.0 effort=20 velocity=50
- joint thigh_joint_left_2: limit lower=-0.5 upper=0.5 effort=0 velocity=50 -> lower=-1.0 upper=1.0 effort=0 velocity=50
- joint thigh_joint_right_1: limit lower=-0.5 upper=0.5 effort=20 velocity=50 -> lower=-1.0 upper=1.0 effort=20 velocity=50
- joint thigh_joint_right_2: limit lower=-0.5 upper=0.5 effort=0 velocity=50 -> lower=-1.0 upper=1.0 effort=0 velocity=50
