Commit message: update config robot

File: source/isaaclab_assets/isaaclab_assets/legged_v3/cad/robot_urdf/urdf/robot.SLDASM.urdf (robot description, URDF)
Before this commit: robot robot.SLDASM, 11 links, 10 joints
Links:
- link base_link: geometry collision box size=0.44 0.20 0.22; visual mesh filename=../meshes/base_link.STL
- link left_foot_link: geometry collision cylinder length=0.045 radius=0.0765; visual mesh filename=../meshes/left_foot_link.STL
- link left_shin_link_B1: geometry collision box size=0.18 0.013 0.054; visual mesh filename=../meshes/left_shin_link_B1.STL
- link left_shin_link_B2: geometry collision box size=0.18 0.013 0.054; visual mesh filename=../meshes/left_shin_link_B2.STL
- link left_thigh_link_A1: geometry collision box size=0.14 0.013 0.048; visual mesh filename=../meshes/left_thigh_link_A1.STL
- link left_thigh_link_A2: geometry collision box size=0.14 0.013 0.048; visual mesh filename=../meshes/left_thigh_link_A2.STL
- link right_foot_link: geometry collision cylinder length=0.045 radius=0.0765; visual mesh filename=../meshes/right_foot_link.STL
- link right_shin_link_B1: geometry collision box size=0.18 0.013 0.054; visual mesh filename=../meshes/right_shin_link_B1.STL
- link right_shin_link_B2: geometry collision box size=0.18 0.013 0.054; visual mesh filename=../meshes/right_shin_link_B2.STL
- link right_thigh_link_A1: geometry collision box size=0.14 0.013 0.048; visual mesh filename=../meshes/right_thigh_link_A1.STL
- link right_thigh_link_A2: mass 0 -> 0.116525440310417; geometry collision box size=0.14 0.013 0.048; visual mesh filename=../meshes/right_thigh_link_A2.STL
Joints:
- joint left_hip_joint_A1: limit lower=0 upper=0 effort=0 velocity=0 -> lower=-1.0 upper=1.0 effort=20 velocity=50
- joint left_hip_joint_A2: limit lower=0 upper=0 effort=0 velocity=0 -> lower=-1.0 upper=1.0 effort=0 velocity=50
- joint left_knee_joint_B1: limit lower=0 upper=0 effort=0 velocity=0 -> lower=-1.0 upper=1.0 effort=20 velocity=50
- joint left_knee_joint_B2: limit lower=0 upper=0 effort=0 velocity=0 -> lower=-1.0 upper=1.0 effort=0 velocity=50
- joint right_hip_joint_A1: limit lower=0 upper=0 effort=0 velocity=0 -> lower=-1.0 upper=1.0 effort=20 velocity=50
- joint right_hip_joint_A2: limit lower=0 upper=0 effort=0 velocity=0 -> lower=-1.0 upper=1.0 effort=0 velocity=50
- joint right_knee_joint_B1: limit lower=0 upper=0 effort=0 velocity=0 -> lower=-1.0 upper=1.0 effort=20 velocity=50
- joint right_knee_joint_B2: limit lower=0 upper=0 effort=0 velocity=0 -> lower=-1.0 upper=1.0 effort=0 velocity=50

Commit message: update stl

File: source/isaaclab_assets/isaaclab_assets/legged_v3/cad/robot_urdf/urdf/robot.SLDASM.urdf (robot description, URDF)
Before this commit: robot robot.SLDASM, 11 links, 10 joints
Joints:
- joint left_hip_joint_A1: limit lower=-1.0 upper=1.0 effort=20 velocity=50 -> lower=-2.0944 upper=2.0944 effort=20 velocity=50
- joint left_hip_joint_A2: limit lower=-1.0 upper=1.0 effort=0 velocity=50 -> lower=-2.0944 upper=2.0944 effort=0 velocity=50
- joint left_knee_joint_B1: limit lower=-1.0 upper=1.0 effort=20 velocity=50 -> lower=-2.0944 upper=2.0944 effort=20 velocity=50
- joint left_knee_joint_B2: limit lower=-1.0 upper=1.0 effort=0 velocity=50 -> lower=-2.0944 upper=2.0944 effort=0 velocity=50
- joint right_hip_joint_A1: limit lower=-1.0 upper=1.0 effort=20 velocity=50 -> lower=-2.0944 upper=2.0944 effort=20 velocity=50
- joint right_hip_joint_A2: limit lower=-1.0 upper=1.0 effort=0 velocity=50 -> lower=-2.0944 upper=2.0944 effort=0 velocity=50
- joint right_knee_joint_B1: limit lower=-1.0 upper=1.0 effort=20 velocity=50 -> lower=-2.0944 upper=2.0944 effort=20 velocity=50
- joint right_knee_joint_B2: limit lower=-1.0 upper=1.0 effort=0 velocity=50 -> lower=-2.0944 upper=2.0944 effort=0 velocity=50

Commit message: update mesh

File: source/isaaclab_assets/isaaclab_assets/legged_v3/cad/robot_urdf/urdf/robot.SLDASM.urdf (robot description, URDF)
Before this commit: robot robot.SLDASM, 11 links, 10 joints
Links:
- link base_link: mass 7.3226 -> 9.2985458095
- link left_foot_link: mass 0.234111484545512 -> 0.2960462476
- link left_shin_link_B1: mass 0.142525440310417 -> 0.1805684146
- link left_shin_link_B2: mass 0.142525440310417 -> 0.1805684109
- link left_thigh_link_A1: mass 0.116525440310417 -> 0.1476182766
- link left_thigh_link_A2: mass 0.116525440310417 -> 0.1476182766
- link right_foot_link: mass 0.234111484545512 -> 0.2960462542
- link right_shin_link_B1: mass 0.142525440310417 -> 0.1805684109
- link right_shin_link_B2: mass 0.142525440310417 -> 0.1805684146
- link right_thigh_link_A1: mass 0.116525440310417 -> 0.1476182736
- link right_thigh_link_A2: mass 0.116525440310417 -> 0.1476182736
Joints:
- joint left_hip_joint_A1: limit lower=-2.0944 upper=2.0944 effort=20 velocity=50 -> lower=-0.6 upper=0.6 effort=20 velocity=50
- joint left_hip_joint_A2: limit lower=-2.0944 upper=2.0944 effort=0 velocity=50 -> lower=-0.6 upper=0.6 effort=0 velocity=50
- joint left_knee_joint_B1: limit lower=-2.0944 upper=2.0944 effort=20 velocity=50 -> lower=-0.6 upper=0.6 effort=20 velocity=50
- joint left_knee_joint_B2: limit lower=-2.0944 upper=2.0944 effort=0 velocity=50 -> lower=-0.6 upper=0.6 effort=0 velocity=50
- joint right_hip_joint_A1: limit lower=-2.0944 upper=2.0944 effort=20 velocity=50 -> lower=-0.6 upper=0.6 effort=20 velocity=50
- joint right_hip_joint_A2: limit lower=-2.0944 upper=2.0944 effort=0 velocity=50 -> lower=-0.6 upper=0.6 effort=0 velocity=50
- joint right_knee_joint_B1: limit lower=-2.0944 upper=2.0944 effort=20 velocity=50 -> lower=-0.6 upper=0.6 effort=20 velocity=50
- joint right_knee_joint_B2: limit lower=-2.0944 upper=2.0944 effort=0 velocity=50 -> lower=-0.6 upper=0.6 effort=0 velocity=50

Commit message: update temp urdf + methodology

File: source/isaaclab_assets/isaaclab_assets/legged_v3/cad/robot_urdf/urdf/robot.SLDASM.urdf (robot description, URDF)
Before this commit: robot robot.SLDASM, 11 links, 10 joints
Links:
- link base_link: mass 9.2985458095 -> 4.6492729048; geometry collision box size=0.35 0.2 0.2; visual mesh filename=../meshes/base_link.STL
- link left_shin_link_B1: geometry collision box size=0.18 0.025 0.025; visual mesh filename=../meshes/left_shin_link_B1.STL
- link left_shin_link_B2: geometry collision box size=0.18 0.025 0.025; visual mesh filename=../meshes/left_shin_link_B2.STL
- link left_thigh_link_A1: geometry collision box size=0.14 0.025 0.025; visual mesh filename=../meshes/left_thigh_link_A1.STL
- link left_thigh_link_A2: geometry collision box size=0.14 0.025 0.025; visual mesh filename=../meshes/left_thigh_link_A2.STL
- link right_shin_link_B1: geometry collision box size=0.18 0.025 0.025; visual mesh filename=../meshes/right_shin_link_B1.STL
- link right_shin_link_B2: geometry collision box size=0.18 0.025 0.025; visual mesh filename=../meshes/right_shin_link_B2.STL
- link right_thigh_link_A1: geometry collision box size=0.14 0.025 0.025; visual mesh filename=../meshes/right_thigh_link_A1.STL
- link right_thigh_link_A2: geometry collision box size=0.14 0.025 0.025; visual mesh filename=../meshes/right_thigh_link_A2.STL
Joints:
- joint left_hip_joint_A1: limit lower=-0.6 upper=0.6 effort=20 velocity=50 -> lower=-0.7745 upper=0.7745 effort=20 velocity=50
- joint left_hip_joint_A2: limit lower=-0.6 upper=0.6 effort=0 velocity=50 -> lower=-0.7745 upper=0.7745 effort=0 velocity=50
- joint left_knee_joint_B1: limit lower=-0.6 upper=0.6 effort=20 velocity=50 -> lower=-0.7745 upper=0.7745 effort=20 velocity=50
- joint left_knee_joint_B2: limit lower=-0.6 upper=0.6 effort=0 velocity=50 -> lower=-0.7745 upper=0.7745 effort=0 velocity=50
- joint right_hip_joint_A1: limit lower=-0.6 upper=0.6 effort=20 velocity=50 -> lower=-0.7745 upper=0.7745 effort=20 velocity=50
- joint right_hip_joint_A2: limit lower=-0.6 upper=0.6 effort=0 velocity=50 -> lower=-0.7745 upper=0.7745 effort=0 velocity=50
- joint right_knee_joint_B1: limit lower=-0.6 upper=0.6 effort=20 velocity=50 -> lower=-0.7745 upper=0.7745 effort=20 velocity=50
- joint right_knee_joint_B2: limit lower=-0.6 upper=0.6 effort=0 velocity=50 -> lower=-0.7745 upper=0.7745 effort=0 velocity=50
